Commit message: feat(t4): 移植 PHP 翻箱 mimic 配方为 t4_vault_mimic 任务
- t4_std.urdf 并入 spherehand 手部碰撞与质量（翻箱撑手必需，fixed joint 合并进 AL7/AR7）
- vault_mimic 包：MotionCommand RSI/adaptive sampling、tracking 奖励/终止、Stage E plant + 0.25 scale
- 训练入口走 gym + legacy RSL-RL wrapper，超参沿用已证 PHP 配方
- 纯 Python 合同测试锁定 manifest/URDF/scale 一致性

Co-authored-by: Cursor <cursoragent@cursor.com>

File: legged_lab/assets/t4/urdf/t4_std.urdf (robot description, URDF)
Before this commit: robot T4, 30 links, 29 joints
Links:
- added link left_sphere_hand_link, mass 0.124; collision mesh filename=../meshes/half_sphere.obj; visual mesh filename=../meshes/half_sphere.obj
- added link left_sphere_hand_tip_link; collision sphere radius=0.001; visual sphere radius=0.001
- added link right_sphere_hand_link, mass 0.124; collision mesh filename=../meshes/half_sphere.obj; visual mesh filename=../meshes/half_sphere.obj
- added link right_sphere_hand_tip_link; collision sphere radius=0.001; visual sphere radius=0.001
Joints:
- added joint left_hand_palm_joint: type fixed, parent AL7, child left_sphere_hand_link, origin xyz=0 0 -0.031 rpy=0 3.14159265359 0
- added joint left_sphere_hand_tip_joint: type fixed, parent left_sphere_hand_link, child left_sphere_hand_tip_link, origin xyz=0 0 0.03 rpy=0 0 0
- added joint right_hand_palm_joint: type fixed, parent AR7, child right_sphere_hand_link, origin xyz=0 0 -0.031 rpy=0 3.14159265359 0
- added joint right_sphere_hand_tip_joint: type fixed, parent right_sphere_hand_link, child right_sphere_hand_tip_link, origin xyz=0 0 0.03 rpy=0 0 0
