Commit message: 修复T4小腿胶囊自碰并冻结污染训练

File: legged_lab/assets/t4/urdf/t4_std.urdf (robot description, URDF)
Before this commit: robot T4, 34 links, 33 joints
Links:
- link Shank_Left: geometry collision cylinder length=0.1 radius=0.05; collision cylinder length=0.20 radius=0.04
- link Shank_Right: geometry collision cylinder length=0.1 radius=0.05; collision cylinder length=0.20 radius=0.04
- link Trunk: geometry collision box size=0.10 0.16 0.34; visual mesh filename=../meshes/head_yaw_link.stl scale=0.001 0.001 0.001
